Commit message: updated config

File: ilab_ur_description/srdf/flexicart.xacro (robot description, xacro)
@@ -1,5 +1,5 @@
 <?xml version="1.0" ?>
 <robot xmlns:xacro="http://www.ros.org/wiki/xacro">
-  <xacro:macro name="flexicart" params="arm_id:='ur' ">
+  <xacro:macro name="ur_flexicart" params="arm_id:='ur' ">
     <disable_collisions link1="${arm_id}_flexicart" link2="base_link" reason="Adjacent"/>
     <disable_collisions link1="${arm_id}_flexicart" link2="base_link_inertia" reason="Adjacent"/>

File: ilab_ur_description/srdf/ilab_ur.srdf.xacro (robot description, xacro)
@@ -8,4 +8,4 @@
   <xacro:include filename="$(find ilab_ur_description)/srdf/flexicart.xacro" />
   <xacro:ilab_ur_macro name="$(arg name)" prefix="$(arg prefix)" />
-  <xacro:flexicart/>
+  <xacro:ur_flexicart/>
 </robot>

File: ilab_ur_description/urdf/flexicart.xacro (robot description, xacro)
@@ -10,5 +10,5 @@
       </joint>
     </xacro:unless>
-    <material name="Gray">
+    <material name="${ns}_gray">
       <color rgba="${125/255} ${125/255} ${125/255} 1.0"/>
     </material>
@@ -19,5 +19,5 @@
           <mesh filename="file://$(find ilab_ur_description)/meshes/flexicart.stl"/>
         </geometry>
-        <material name="Gray"/>
+        <material name="${ns}_gray"/>
       </visual>
       <collision>
